File: Misc - Mounting Holes.kicad_sch (KiCad schematic)
At the start: 0 parts

Commit message: Added footprints, images, almost finished all èages except for the MCU
Parts:
- added C2801, C2802, C2803, C2804: 1n X7R 1kV, Capacitor_SMD:C_0603_1608Metric, symbol Device:C_Small
- added FM2801, FM2802, FM2803: Fiducial, Charge_Manager_FP:Fiducial_1mm_Mask2mm, symbol Mechanical:Fiducial
- added H2801, H2802, H2803, H2804: M2.5 (2.7mm), MountingHole:MountingHole_2.5mm_Pad_Via, symbol Mechanical:MountingHole_Pad
- added R2801, R2802, R2803, R2804: 0R 1%, Resistor_SMD:R_0603_1608Metric, symbol Device:R
Connections:
- new net GND: C2801.2, C2802.2, C2803.2, C2804.2, R2801.2, R2802.2, R2803.2, R2804.2
- new net HOLE1: C2801.1, H2801.1, R2801.1
- new net HOLE2: C2802.1, C2803.1, H2802.1, H2803.1, R2802.1, R2803.1
- new net HOLE4: C2804.1, H2804.1, R2804.1
Other:
- note added: "How to connect mounting holes."
- note added: "Inspired by Amulet controller Schematics by Vincent Nguyen"
- note added: "PCB Mounting Holes"
- title: (none) -> Misc - Mounting Holes & Fiducials
