File: Plume.kicad_pcb (KiCad board)
At the start: 6 copper layers, 70 x 40 mm, 395 parts, among them IC1001 DRV8214RTER, IC1101 DRV8214RTER, IC1201 DRV8214RTER, IC1301 DRV8214RTER, IC1401 DRV8214RTER, IC1501 DRV8214RTER, IC1601 DRV8214RTER, IC1701 DRV8214RTER, IC1801 DRV8214RTER, IC1901 DRV8214RTER, IC2001 DRV8214RTER, IC2101 DRV8214RTER, IC2201 DRV8214RTER, IC2301 DRV8214RTER, IC2401 DRV8214RTER, IC2501 DRV8214RTER, IC2601 DRV8214RTER, IC2701 DRV8214RTER, IC2801 SN74AHCT1G125DRLR, IC2802 REG71050DRVT, J401 Solder Holes 4x1 2.54mm 22AWG, J402 Conn_ARM_SWD_TagConnect_TC203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, J403 Solder Wire Pad 2x4mm, J404 Solder Wire Pad 2x4mm, J501 S2B-PH-SM4-TB, J601 USB_C_Receptacle_PowerOnly_6P, J602 Solder Wire Pad 2x4mm, J603 Solder Wire Pad 2x4mm, J901 SEI-125-02-GF-S-M-AT, J902 SEI-115-02-GF-S-M-AT, Q501 NMOS IRLML6344TRPBF SOT-23, Q502 CSD85302L, Q601 CSD75207W15, Q701 PMOS SI2365EDS-T1-GE3, SW401 KMR232NG ULC, SW402 KMR232NG ULC, SW403 CAS-D20A1, SW404 KMR232NG ULC, SW405 KMR232NG ULC, SW406 KMR232NG ULC, SW407 KMR232NG ULC, U401 STM32WB5MMGH6TR, U501 BQ29737DSER, U502 MCP73831T-2ACI/MC, U601 BQ51013CQWRHLRQ1, U701 TPS3839G33DQNR, U702 TPS7A0233DQNR, U801 PCA9546ARGVR

Commit message: Reviewed shematic, cleaned all DRC errors, chosed stackup, started layout
Parts:
- removed J501: S2B-PH-SM4-TB, 0_Plume:CONN_S2B-PH-SM4-TB_JST
- removed LED1001, LED1101, LED1201, LED1301, LED1401, LED1501, LED1601, LED1701, LED1801, LED1901, LED2001, LED2101, LED2201, LED2301, LED2401, LED2501, LED2601, LED2701: BLUE, 0_Plume:KingBright_LED_0603
- removed LED601: RED, 0_Plume:Bivar_LED_0603
- removed TP704: VBAT, 0_Plume:TestPoint_Pad_D0.5mm_Back
- added J502: S2B-PH-SM4-TB, 0_Plume:CONN_S2B-PH-SM4-TB_JST, F.Cu at (131.0, 120.0)
- added LED1002: BLUE, 0_Plume:KingBright_LED_0603, F.Cu at (217.6, 65.7)
- added LED1003: BLUE, 0_Plume:KingBright_LED_0603, F.Cu at (217.6, 60.3)
- added LED1004: BLUE, 0_Plume:KingBright_LED_0603, F.Cu at (193.6, 33.7)
- added LED1005: BLUE, 0_Plume:KingBright_LED_0603, F.Cu at (205.6, 73.6)
- added LED1006: BLUE, 0_Plume:KingBright_LED_0603, F.Cu at (217.6, 33.7)
- added LED1007: BLUE, 0_Plume:KingBright_LED_0603, F.Cu at (193.6, 60.3)
- added LED1008: BLUE, 0_Plume:KingBright_LED_0603, F.Cu at (205.6, 60.3)
- added LED1009: BLUE, 0_Plume:KingBright_LED_0603, F.Cu at (229.5, 33.7)
- added LED1010: BLUE, 0_Plume:KingBright_LED_0603, F.Cu at (193.6, 73.6)
- added LED1011: BLUE, 0_Plume:KingBright_LED_0603, F.Cu at (217.6, 47.0)
- added LED1012: BLUE, 0_Plume:KingBright_LED_0603, F.Cu at (205.6, 33.7)
- added LED1013: BLUE, 0_Plume:KingBright_LED_0603, F.Cu at (229.5, 47.0)
- added LED1014: BLUE, 0_Plume:KingBright_LED_0603, F.Cu at (181.6, 47.0)
- added LED1015: BLUE, 0_Plume:KingBright_LED_0603, F.Cu at (205.6, 47.0)
- added LED1016: BLUE, 0_Plume:KingBright_LED_0603, F.Cu at (181.6, 33.7)
- added LED1017: BLUE, 0_Plume:KingBright_LED_0603, F.Cu at (193.6, 47.0)
- added LED1018: BLUE, 0_Plume:KingBright_LED_0603, F.Cu at (181.6, 60.3)
- added LED1019: BLUE, 0_Plume:KingBright_LED_0603, F.Cu at (181.6, 73.6)
- added LED602: RED, 0_Plume:Bivar_LED_0603, F.Cu at (217.6, 70.2)
- C1101, C1102, C1103, C1201, C1202, C1203, C1301, C1302, C1303, C1401, C1402, C1403, C1501, C1502, C1503, C1601, C1602, C1603, C1701, C1702, C1703, C1801, C1802, C1803, C1901, C1902, C1903, C2001, C2002, C2003, C2101, C2102, C2103, C2201, C2202, C2203, C2301, C2302, C2303, C2401, C2402, C2403, C2501, C2502, C2503, C2601, C2602, C2603, C2701, C2702, C2703, IC1101, IC1201, IC1301, IC1401, IC1501, IC1601, IC1701, IC1801, IC1901, IC2001, IC2101, IC2201, IC2301, IC2401, IC2501, IC2601, IC2701, R1101, R1102, R1103, R1201, R1202, R1203, R1301, R1302, R1303, R1401, R1402, R1403, R1501, R1502, R1503, R1601, R1602, R1603, R1701, R1702, R1703, R1801, R1802, R1803, R1901, R1902, R1903, R2001, R2002, R2003, R2101, R2102, R2103, R2201, R2202, R2203, R2301, R2302, R2303, R2401, R2402, R2403, R2501, R2502, R2503, R2601, R2602, R2603, R2701, R2702, R2703, TP1101, TP1102, TP1103, TP1104, TP1201, TP1202, TP1203, TP1204, TP1301, TP1302, TP1303, TP1304, TP1401, TP1402, TP1403, TP1404, TP1501, TP1502, TP1503, TP1504, TP1601, TP1602, TP1603, TP1604, TP1701, TP1702, TP1703, TP1704, TP1801, TP1802, TP1803, TP1804, TP1901, TP1902, TP1903, TP1904, TP2001, TP2002, TP2003, TP2004, TP2101, TP2102, TP2103, TP2104, TP2201, TP2202, TP2203, TP2204, TP2301, TP2302, TP2303, TP2304, TP2401, TP2402, TP2403, TP2404, TP2501, TP2502, TP2503, TP2504, TP2601, TP2602, TP2603, TP2604, TP2701, TP2702, TP2703, TP2704: moved to F.Cu
- J602, J603: footprint 0_Plume:SolderWirePad_SMD_2x4mm -> 0_Plume:SolderWirePad_SMD_1,5x3mm
- TP701: value COUT -> 3V3_EN
- TP702: value DOUT -> +3V3
- TP703: value -VBAT -> +VDD
- U601: footprint 0_Plume:BQ51013CQWRHLRQ1 -> Package_DFN_QFN:Texas_VQFN-RHL-20
- moved TP2101 142.3 mm to (233.6, 38.7)
- moved TP2103 141.9 mm to (235.2, 38.7)
- moved TP2102 140.6 mm to (233.6, 40.3)
- moved TP2104 140.2 mm to (235.2, 40.3)
- moved R2101 136.7 mm to (233.0, 44.2)
- moved C2102 135.0 mm to (235.9, 44.2)
- moved C2103 135.0 mm to (235.9, 46.2)
- moved R2102 133.5 mm to (233.0, 46.2)
- moved R2103 133.5 mm to (233.0, 48.2)
- moved IC2101 132.2 mm to (230.2, 40.6)
- moved C2101 127.7 mm to (229.5, 44.5)
- moved TP1701 124.4 mm to (233.6, 25.4)
- moved TP1703 123.6 mm to (235.2, 25.4)
- moved TP1702 122.4 mm to (233.6, 27.0)
- moved TP1704 121.6 mm to (235.2, 27.0)
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Connections:
- net Net-(J601-CC1) renamed /Project Architecture/Power - Wireless Receiver & USB/CC1
- net Net-(J601-CC2) renamed /Project Architecture/Power - Wireless Receiver & USB/CC2
- C2903 pad 1: /Project Architecture/Misc - Mounting Holes & Fiducials/HOLE2 -> /Project Architecture/Misc - Mounting Holes & Fiducials/HOLE3
- H2903 pad 1: /Project Architecture/Misc - Mounting Holes & Fiducials/HOLE2 -> /Project Architecture/Misc - Mounting Holes & Fiducials/HOLE3
- IC2001 pad 10: +3V3 -> /Project Architecture/Motor Control - Drivers/Motor Control - Driver 10/A0
- IC2001 pad 11: /Project Architecture/MCU - Unit/nSLEEP_BACK -> /Project Architecture/MCU - Unit/nSLEEP_FRONT
- IC2101 pad 10: /Project Architecture/Motor Control - Drivers/Motor Control - Driver 11/A0 -> +3V3
- IC2101 pad 11: /Project Architecture/MCU - Unit/nSLEEP_FRONT -> /Project Architecture/MCU - Unit/nSLEEP_REAR
- IC2201 pad 11: /Project Architecture/MCU - Unit/nSLEEP_BACK -> /Project Architecture/MCU - Unit/nSLEEP_REAR
- IC2301 pad 11: /Project Architecture/MCU - Unit/nSLEEP_BACK -> /Project Architecture/MCU - Unit/nSLEEP_REAR
- IC2401 pad 11: /Project Architecture/MCU - Unit/nSLEEP_BACK -> /Project Architecture/MCU - Unit/nSLEEP_REAR
- IC2501 pad 11: /Project Architecture/MCU - Unit/nSLEEP_BACK -> /Project Architecture/MCU - Unit/nSLEEP_REAR
- IC2601 pad 11: /Project Architecture/MCU - Unit/nSLEEP_BACK -> /Project Architecture/MCU - Unit/nSLEEP_REAR
- IC2701 pad 11: /Project Architecture/MCU - Unit/nSLEEP_BACK -> /Project Architecture/MCU - Unit/nSLEEP_REAR
- J901 pad 23: /Project Architecture/Motor Control - Drivers/Motor Control - Driver 11/OUT1 -> /Project Architecture/Motor Control - Drivers/Motor Control - Driver 10/OUT1
- J901 pad 24: /Project Architecture/Motor Control - Drivers/Motor Control - Driver 11/OUT2 -> /Project Architecture/Motor Control - Drivers/Motor Control - Driver 10/OUT2
- J902 pad 1: /Project Architecture/Motor Control - Drivers/Motor Control - Driver 10/OUT1 -> /Project Architecture/Motor Control - Drivers/Motor Control - Driver 11/OUT1
- J902 pad 2: /Project Architecture/Motor Control - Drivers/Motor Control - Driver 10/OUT2 -> /Project Architecture/Motor Control - Drivers/Motor Control - Driver 11/OUT2
- R2903 pad 1: /Project Architecture/Misc - Mounting Holes & Fiducials/HOLE2 -> /Project Architecture/Misc - Mounting Holes & Fiducials/HOLE3
- TP2005 pad 1: +3V3 -> /Project Architecture/Motor Control - Drivers/Motor Control - Driver 10/A0
- TP2105 pad 1: /Project Architecture/Motor Control - Drivers/Motor Control - Driver 11/A0 -> +3V3
- TP701 pad 1: /Project Architecture/Power - Path & Generation/COUT -> /Project Architecture/Power - Path & Generation/3V3_EN
- TP702 pad 1: /Project Architecture/Power - Path & Generation/DOUT -> +3V3
- TP703 pad 1: /Project Architecture/Power - Path & Generation/-VBAT -> /Project Architecture/Power - Path & Generation/+VDD
- TP902 pad 1: /Project Architecture/MCU - Unit/nSLEEP_BACK -> /Project Architecture/MCU - Unit/nSLEEP_REAR
- U401 pad 11: /Project Architecture/MCU - Unit/I2C1_SDA -> /Project Architecture/Logic - I2C Mux/I2C1_SDA
- U401 pad 14: /Project Architecture/MCU - Unit/I2C1_SCL -> /Project Architecture/Logic - I2C Mux/I2C1_SCL
- U401 pad 39: /Project Architecture/Motor Control - Drivers/Motor Control - Driver 10/nFAULT -> /Project Architecture/Motor Control - Drivers/Motor Control - Driver 11/nFAULT
- U401 pad 40: /Project Architecture/Motor Control - Drivers/Motor Control - Driver 11/nFAULT -> /Project Architecture/Motor Control - Drivers/Motor Control - Driver 10/nFAULT
- U401 pad 77: unconnected-(U401A-PD10-Pad77) -> /Project Architecture/MCU - Unit/EN1
- U401 pad 82: unconnected-(U401A-PD11-Pad82) -> /Project Architecture/MCU - Unit/EN2
- U601 pad 10: /Project Architecture/Power - Wireless Receiver & USB/EN1 -> /Project Architecture/MCU - Unit/EN1
- U601 pad 11: /Project Architecture/Power - Wireless Receiver & USB/EN2 -> /Project Architecture/MCU - Unit/EN2
- U801 pad 1: GND -> /Project Architecture/Logic - I2C Mux/MUX_RESET
- U801 pad 10: /Project Architecture/Logic - I2C Mux/SD2 -> /Project Architecture/Logic - I2C Mux/SD3
- U801 pad 11: /Project Architecture/Logic - I2C Mux/SC3 -> GND
- U801 pad 12: /Project Architecture/Logic - I2C Mux/SD3 -> /Project Architecture/Logic - I2C Mux/I2C1_SCL
- U801 pad 13: GND -> /Project Architecture/Logic - I2C Mux/I2C1_SDA
- U801 pad 14: /Project Architecture/Logic - I2C Mux/I2C1_SCL -> +3V3
- U801 pad 15: /Project Architecture/Logic - I2C Mux/I2C1_SDA -> GND
- U801 pad 16: +3V3 -> GND
- U801 pad 2: GND -> /Project Architecture/Logic - I2C Mux/SD0
- U801 pad 3: /Project Architecture/Logic - I2C Mux/MUX_RESET -> /Project Architecture/Logic - I2C Mux/SC0
- U801 pad 4: /Project Architecture/Logic - I2C Mux/SD0 -> /Project Architecture/Logic - I2C Mux/SD1
- U801 pad 5: /Project Architecture/Logic - I2C Mux/SC0 -> /Project Architecture/Logic - I2C Mux/SC1
- U801 pad 6: /Project Architecture/Logic - I2C Mux/SD1 -> GND
- U801 pad 7: /Project Architecture/Logic - I2C Mux/SC1 -> /Project Architecture/Logic - I2C Mux/SC2
- U801 pad 8: GND -> /Project Architecture/Logic - I2C Mux/SD2
- U801 pad 9: /Project Architecture/Logic - I2C Mux/SC2 -> /Project Architecture/Logic - I2C Mux/SC3
Other:
- outline, holes or cut-outs redrawn

Commit message: Cleaned repo, cleaned and exported shematic, advanced rough layout
Parts:
- C1101, C1102, C1103, C1201, C1202, C1203, C1301, C1302, C1303, C1401, C1402, C1403, C1501, C1502, C1503, C1601, C1602, C1603, C1701, C1702, C1703, C1801, C1802, C1803, C1901, C1902, C1903, C2001, C2002, C2003, C2101, C2102, C2103, C2201, C2202, C2203, C2301, C2302, C2303, C2401, C2402, C2403, C2501, C2502, C2503, C2601, C2602, C2603, C2701, C2702, C2703, C2904, IC1101, IC1201, IC1301, IC1401, IC1501, IC1601, IC1701, IC1801, IC1901, IC2001, IC2101, IC2201, IC2301, IC2401, IC2501, IC2601, IC2701, R1101, R1102, R1103, R1201, R1202, R1203, R1301, R1302, R1303, R1401, R1402, R1403, R1501, R1502, R1503, R1601, R1602, R1603, R1701, R1702, R1703, R1801, R1802, R1803, R1901, R1902, R1903, R2001, R2002, R2003, R2101, R2102, R2103, R2201, R2202, R2203, R2301, R2302, R2303, R2401, R2402, R2403, R2501, R2502, R2503, R2601, R2602, R2603, R2701, R2702, R2703, R2904, TP1001, TP1002, TP1005, TP1006, TP1101, TP1102, TP1103, TP1104, TP1105, TP1106, TP1201, TP1202, TP1203, TP1204, TP1205, TP1206, TP1301, TP1302, TP1303, TP1304, TP1305, TP1306, TP1401, TP1402, TP1403, TP1404, TP1405, TP1406, TP1501, TP1502, TP1503, TP1504, TP1505, TP1506, TP1601, TP1602, TP1603, TP1604, TP1605, TP1606, TP1701, TP1702, TP1703, TP1704, TP1705, TP1706, TP1801, TP1802, TP1803, TP1804, TP1805, TP1806, TP1901, TP1902, TP1903, TP1904, TP1905, TP1906, TP2001, TP2002, TP2003, TP2004, TP2005, TP2006, TP2101, TP2102, TP2103, TP2104, TP2105, TP2106, TP2201, TP2202, TP2203, TP2204, TP2205, TP2206, TP2301, TP2302, TP2303, TP2304, TP2305, TP2306, TP2401, TP2402, TP2403, TP2404, TP2405, TP2406, TP2501, TP2502, TP2503, TP2504, TP2505, TP2506, TP2601, TP2602, TP2603, TP2604, TP2605, TP2606, TP2701, TP2702, TP2703, TP2704, TP2705, TP2706: moved to B.Cu
- C703: moved to F.Cu
- J403, J404: value Solder Wire Pad 2x4mm -> Solder Wire Pad 1,5x3mm; footprint 0_Plume:SolderWirePad_SMD_2x4mm -> 0_Plume:SolderWirePad_SMD_1,5x3mm
- J602, J603: value Solder Wire Pad 2x4mm -> Solder Wire Pad 1,5x3mm
- LED1001: renamed from LED1002; moved to B.Cu
- LED1101: renamed from LED1003; moved to B.Cu
- LED1201: renamed from LED1004; moved to B.Cu
- LED1301: renamed from LED1005; moved to B.Cu
- LED1401: renamed from LED1006; moved to B.Cu
- LED1501: renamed from LED1007; moved to B.Cu
- LED1601: renamed from LED1008; moved to B.Cu
- LED1701: renamed from LED1009; moved to B.Cu
- LED1801: renamed from LED1010; moved to B.Cu
- LED1901: renamed from LED1011; moved to B.Cu
- LED2001: renamed from LED1012; moved to B.Cu
- LED2101: renamed from LED1013; moved to B.Cu
- LED2201: renamed from LED1014; moved to B.Cu
- LED2301: renamed from LED1015; moved to B.Cu
- LED2401: renamed from LED1016; moved to B.Cu
- LED2501: renamed from LED1017; moved to B.Cu
- LED2601: renamed from LED1018; moved to B.Cu
- LED2701: renamed from LED1019; moved to B.Cu
- U601: footprint Package_DFN_QFN:Texas_VQFN-RHL-20 -> 0_Plume:Texas_VQFN-RHL-20
- moved R2903 135.7 mm to (176.0, 121.8), turned to 180 degrees
- moved R2904 130.4 mm to (122.8, 117.8), turned to 90 degrees
- moved TP1705 112.8 mm to (164.7, 112.2), turned to -90 degrees
- moved SW404 112.4 mm to (168.9, 112.5)
- moved R601 112.4 mm to (127.0, 103.2)
- moved TP1706 111.1 mm to (165.4, 112.2), turned to -90 degrees
- moved C502 111.1 mm to (143.2, 111.5)
- moved Q501 111.1 mm to (143.7, 108.8)
- moved R502 111.1 mm to (139.8, 107.4)
- moved R509 111.1 mm to (139.8, 111.4)
- moved R503 111.1 mm to (139.8, 109.4)
- moved TP1405 110.9 mm to (155.8, 112.2), turned to -90 degrees
- moved TP1005 109.8 mm to (155.7, 122.2), turned to -90 degrees
- moved TP504 109.5 mm to (138.2, 108.5)
- moved TP505 109.5 mm to (138.2, 110.1)
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- renumbered J502 to J501, LED602 to LED601
Connections:
- D401 pad 1: /Project Architecture/MCU - Unit/USART1_TX -> /Project Architecture/MCU - Unit/USART1_RX
- D401 pad 3: /Project Architecture/MCU - Unit/USART1_RX -> /Project Architecture/MCU - Unit/USART1_TX

Commit message: Advanced rough layout
Parts:
- removed C702: 1u X7R 16V, Capacitor_SMD:C_0603_1608Metric
- removed LED601: RED, 0_Plume:Bivar_LED_0603
- removed R402: 5k1 1%, Resistor_SMD:R_0402_1005Metric
- removed R601: 680R 1%, Resistor_SMD:R_0402_1005Metric
- added C2805: 100n X7R 16V, Capacitor_SMD:C_0402_1005Metric, F.Cu at (138.5, 102.0)
- added C2806: 100n X7R 16V, Capacitor_SMD:C_0402_1005Metric, F.Cu at (136.5, 102.0)
- added C404: 100n X7R 16V, Capacitor_SMD:C_0402_1005Metric, F.Cu at (153.2, 110.2)
- added C405: 100n X7R 16V, Capacitor_SMD:C_0402_1005Metric, F.Cu at (153.2, 114.5)
- added C406: 100n X7R 16V, Capacitor_SMD:C_0402_1005Metric, F.Cu at (153.2, 118.8)
- added C407: 100n X7R 16V, Capacitor_SMD:C_0402_1005Metric, F.Cu at (153.2, 123.0)
- added C408: 3p3 C0G 50V, Capacitor_SMD:C_0402_1005Metric, F.Cu at (183.0, 135.1)
- added C409: 3p3 C0G 50V, Capacitor_SMD:C_0402_1005Metric, F.Cu at (183.0, 137.0)
- added C410: 3p3 C0G 50V, Capacitor_SMD:C_0402_1005Metric, F.Cu at (183.0, 139.0)
- added C506: 47u X5R 16V, Capacitor_SMD:C_1206_3216Metric, F.Cu at (126.2, 116.8)
- added C507: 47u X5R 16V, Capacitor_SMD:C_1206_3216Metric, F.Cu at (123.9, 116.8)
- added C617: 10u X5R 16V, Capacitor_SMD:C_0603_1608Metric, F.Cu at (134.0, 92.8)
- added C618: 10u X5R 16V, Capacitor_SMD:C_0603_1608Metric, F.Cu at (135.5, 92.8)
- added C704: 10u X5R 16V, Capacitor_SMD:C_0603_1608Metric, F.Cu at (124.4, 106.6)
- added J405: Solder Wire Pad 1,5x3mm, 0_Plume:SolderWirePad_SMD_1,5x3mm, F.Cu at (128.8, 112.8)
- added J406: Solder Wire Pad 1,5x3mm, 0_Plume:SolderWirePad_SMD_1,5x3mm, F.Cu at (135.2, 112.8)
- added J407: Solder Wire Pad 1,5x3mm, 0_Plume:SolderWirePad_SMD_1,5x3mm, B.Cu at (150.5, 86.8)
- added J408: Solder Wire Pad 1,5x3mm, 0_Plume:SolderWirePad_SMD_1,5x3mm, B.Cu at (148.2, 86.8)
- added J604: Solder Wire Pad 1,5x3mm, 0_Plume:SolderWirePad_SMD_1,5x3mm, B.Cu at (131.0, 86.8)
- added J605: Solder Wire Pad 1,5x3mm, 0_Plume:SolderWirePad_SMD_1,5x3mm, B.Cu at (126.0, 86.8)
- added LED502: GREEN, 0_Plume:KingBright_LED_0603, F.Cu at (125.2, 96.5)
- added R510: 330R 1%, Resistor_SMD:R_0402_1005Metric, F.Cu at (125.2, 95.2)
- added R609: 10k 1%, Resistor_SMD:R_0402_1005Metric, F.Cu at (152.5, 93.0)
- added R812: 3k 1%, Resistor_SMD:R_0402_1005Metric, F.Cu at (135.8, 97.5)
- added R813: 3k 1%, Resistor_SMD:R_0402_1005Metric, F.Cu at (137.8, 97.5)
- added TP2807: INT1, 0_Plume:TestPoint_Pad_D0.5mm_Back, F.Cu at (149.5, 81.6)
- added TP2808: INT2, 0_Plume:TestPoint_Pad_D0.5mm_Back, F.Cu at (149.5, 83.1)
- added U3202: BMI270, Package_LGA:Bosch_LGA-14_3x2.5mm_P0.5mm, F.Cu at (137.0, 99.8)
- C1002, C1102, C1202, C1302, C1402, C1502, C1602, C1702, C1802, C1902, C2002, C2102, C2202, C2302, C2402, C2502, C2602, C2702: value 100n X7R 16V -> 100n X7R 50V; footprint Capacitor_SMD:C_0402_1005Metric -> Capacitor_SMD:C_0603_1608Metric
- C2901, R2901: moved to B.Cu
- C607, C613: value 470n X7R 25V -> 470n X5R 25V; footprint Capacitor_SMD:C_0603_1608Metric -> Capacitor_SMD:C_0402_1005Metric
- R508: value 5k1 1% -> 2k2 1%
- TP2803: value DIN_5V -> INT1
- TP2804: value +5V -> INT2
- U702: value TPS7A0233DQNR -> TPS7A0233DBVR; footprint Package_SON:Texas_X2SON-4_1x1mm_P0.65mm -> Package_TO_SOT_SMD:SOT-23-5
- moved C2101 76.7 mm to (245.2, 97.9)
- moved C2102 76.7 mm to (244.0, 97.9)
- moved LED2601 76.5 mm to (251.5, 93.2)
- moved C1001 76.4 mm to (235.8, 117.3)
- moved C1002 76.4 mm to (234.6, 117.3)
- moved C1003 76.4 mm to (230.6, 114.8)
- moved C1101 76.4 mm to (244.4, 117.4)
- moved C1102 76.4 mm to (243.2, 117.4)
- moved C1103 76.4 mm to (239.2, 114.9)
- moved C1201 76.4 mm to (218.1, 107.9)
- moved C1202 76.4 mm to (216.9, 107.9)
- moved C1203 76.4 mm to (212.9, 105.4)
- moved C1301 76.4 mm to (226.9, 117.6)
- moved C1302 76.4 mm to (225.6, 117.6)
- moved C1303 76.4 mm to (221.6, 115.2)
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Connections:
- net /Project Architecture/Motor Control - Drivers/Motor Control - Driver 0/OUT1 renamed /Project Architecture/Motor Control - Drivers/OUT1_0
- net /Project Architecture/Motor Control - Drivers/Motor Control - Driver 0/OUT2 renamed /Project Architecture/Motor Control - Drivers/OUT2_0
- net /Project Architecture/Motor Control - Drivers/Motor Control - Driver 0/nFAULT renamed /Project Architecture/MCU - Unit/nFault0
- net /Project Architecture/Motor Control - Drivers/Motor Control - Driver 1/OUT1 renamed /Project Architecture/Motor Control - Drivers/OUT1_1
- net /Project Architecture/Motor Control - Drivers/Motor Control - Driver 1/OUT2 renamed /Project Architecture/Motor Control - Drivers/OUT2_1
- net /Project Architecture/Motor Control - Drivers/Motor Control - Driver 1/nFAULT renamed /Project Architecture/MCU - Unit/nFault1
- net /Project Architecture/Motor Control - Drivers/Motor Control - Driver 10/OUT1 renamed /Project Architecture/Motor Control - Drivers/OUT1_10
- net /Project Architecture/Motor Control - Drivers/Motor Control - Driver 10/OUT2 renamed /Project Architecture/Motor Control - Drivers/OUT2_10
- net /Project Architecture/Motor Control - Drivers/Motor Control - Driver 10/nFAULT renamed /Project Architecture/MCU - Unit/nFault10
- net /Project Architecture/Motor Control - Drivers/Motor Control - Driver 11/OUT1 renamed /Project Architecture/Motor Control - Drivers/OUT1_11
- net /Project Architecture/Motor Control - Drivers/Motor Control - Driver 11/OUT2 renamed /Project Architecture/Motor Control - Drivers/OUT2_11
- net /Project Architecture/Motor Control - Drivers/Motor Control - Driver 11/nFAULT renamed /Project Architecture/MCU - Unit/nFault11
- net /Project Architecture/Motor Control - Drivers/Motor Control - Driver 12/OUT1 renamed /Project Architecture/Motor Control - Drivers/OUT1_12
- net /Project Architecture/Motor Control - Drivers/Motor Control - Driver 12/OUT2 renamed /Project Architecture/Motor Control - Drivers/OUT2_12
- net /Project Architecture/Motor Control - Drivers/Motor Control - Driver 12/nFAULT renamed /Project Architecture/MCU - Unit/nFault12
- net /Project Architecture/Motor Control - Drivers/Motor Control - Driver 13/OUT1 renamed /Project Architecture/Motor Control - Drivers/OUT1_13
- net /Project Architecture/Motor Control - Drivers/Motor Control - Driver 13/OUT2 renamed /Project Architecture/Motor Control - Drivers/OUT2_13
- net /Project Architecture/Motor Control - Drivers/Motor Control - Driver 13/nFAULT renamed /Project Architecture/MCU - Unit/nFault13
- net /Project Architecture/Motor Control - Drivers/Motor Control - Driver 14/OUT1 renamed /Project Architecture/Motor Control - Drivers/OUT1_14
- net /Project Architecture/Motor Control - Drivers/Motor Control - Driver 14/OUT2 renamed /Project Architecture/Motor Control - Drivers/OUT2_14
- net /Project Architecture/Motor Control - Drivers/Motor Control - Driver 14/nFAULT renamed /Project Architecture/MCU - Unit/nFault14
- net /Project Architecture/Motor Control - Drivers/Motor Control - Driver 15/OUT1 renamed /Project Architecture/Motor Control - Drivers/OUT1_15
- net /Project Architecture/Motor Control - Drivers/Motor Control - Driver 15/OUT2 renamed /Project Architecture/Motor Control - Drivers/OUT2_15
- net /Project Architecture/Motor Control - Drivers/Motor Control - Driver 15/nFAULT renamed /Project Architecture/MCU - Unit/nFault15
- net /Project Architecture/Motor Control - Drivers/Motor Control - Driver 16/OUT1 renamed /Project Architecture/Motor Control - Drivers/OUT1_16
- net /Project Architecture/Motor Control - Drivers/Motor Control - Driver 16/OUT2 renamed /Project Architecture/Motor Control - Drivers/OUT2_16
- net /Project Architecture/Motor Control - Drivers/Motor Control - Driver 16/nFAULT renamed /Project Architecture/MCU - Unit/nFault16
- net /Project Architecture/Motor Control - Drivers/Motor Control - Driver 17/OUT1 renamed /Project Architecture/Motor Control - Drivers/OUT1_17
- net /Project Architecture/Motor Control - Drivers/Motor Control - Driver 17/OUT2 renamed /Project Architecture/Motor Control - Drivers/OUT2_17
- net /Project Architecture/Motor Control - Drivers/Motor Control - Driver 17/nFAULT renamed /Project Architecture/MCU - Unit/nFault17
- net /Project Architecture/Motor Control - Drivers/Motor Control - Driver 2/OUT1 renamed /Project Architecture/Motor Control - Drivers/OUT1_2
- net /Project Architecture/Motor Control - Drivers/Motor Control - Driver 2/OUT2 renamed /Project Architecture/Motor Control - Drivers/OUT2_2
- net /Project Architecture/Motor Control - Drivers/Motor Control - Driver 2/nFAULT renamed /Project Architecture/MCU - Unit/nFault2
- net /Project Architecture/Motor Control - Drivers/Motor Control - Driver 3/OUT1 renamed /Project Architecture/Motor Control - Drivers/OUT1_3
- net /Project Architecture/Motor Control - Drivers/Motor Control - Driver 3/OUT2 renamed /Project Architecture/Motor Control - Drivers/OUT2_3
- net /Project Architecture/Motor Control - Drivers/Motor Control - Driver 3/nFAULT renamed /Project Architecture/MCU - Unit/nFault3
- net /Project Architecture/Motor Control - Drivers/Motor Control - Driver 4/OUT1 renamed /Project Architecture/Motor Control - Drivers/OUT1_4
- net /Project Architecture/Motor Control - Drivers/Motor Control - Driver 4/OUT2 renamed /Project Architecture/Motor Control - Drivers/OUT2_4
- net /Project Architecture/Motor Control - Drivers/Motor Control - Driver 4/nFAULT renamed /Project Architecture/MCU - Unit/nFault4
- net /Project Architecture/Motor Control - Drivers/Motor Control - Driver 5/OUT1 renamed /Project Architecture/Motor Control - Drivers/OUT1_5
- net /Project Architecture/Motor Control - Drivers/Motor Control - Driver 5/OUT2 renamed /Project Architecture/Motor Control - Drivers/OUT2_5
- net /Project Architecture/Motor Control - Drivers/Motor Control - Driver 5/nFAULT renamed /Project Architecture/MCU - Unit/nFault5
- net /Project Architecture/Motor Control - Drivers/Motor Control - Driver 6/OUT1 renamed /Project Architecture/Motor Control - Drivers/OUT1_6
- net /Project Architecture/Motor Control - Drivers/Motor Control - Driver 6/OUT2 renamed /Project Architecture/Motor Control - Drivers/OUT2_6
- net /Project Architecture/Motor Control - Drivers/Motor Control - Driver 6/nFAULT renamed /Project Architecture/MCU - Unit/nFault6
- net /Project Architecture/Motor Control - Drivers/Motor Control - Driver 7/OUT1 renamed /Project Architecture/Motor Control - Drivers/OUT1_7
- net /Project Architecture/Motor Control - Drivers/Motor Control - Driver 7/OUT2 renamed /Project Architecture/Motor Control - Drivers/OUT2_7
- net /Project Architecture/Motor Control - Drivers/Motor Control - Driver 7/nFAULT renamed /Project Architecture/MCU - Unit/nFault7
- net /Project Architecture/Motor Control - Drivers/Motor Control - Driver 8/OUT1 renamed /Project Architecture/Motor Control - Drivers/OUT1_8
- net /Project Architecture/Motor Control - Drivers/Motor Control - Driver 8/OUT2 renamed /Project Architecture/Motor Control - Drivers/OUT2_8
- net /Project Architecture/Motor Control - Drivers/Motor Control - Driver 8/nFAULT renamed /Project Architecture/MCU - Unit/nFault8
- net /Project Architecture/Motor Control - Drivers/Motor Control - Driver 9/OUT1 renamed /Project Architecture/Motor Control - Drivers/OUT1_9
- net /Project Architecture/Motor Control - Drivers/Motor Control - Driver 9/OUT2 renamed /Project Architecture/Motor Control - Drivers/OUT2_9
- net /Project Architecture/Motor Control - Drivers/Motor Control - Driver 9/nFAULT renamed /Project Architecture/MCU - Unit/nFault9
- net Net-(IC2802-CPUMP+) renamed /Project Architecture/User - RGB LED Indicator/CPUMP+
- net Net-(IC2802-C_PUMP-) renamed /Project Architecture/User - RGB LED Indicator/CPUMP-
- net Net-(LED1001-A) renamed /Project Architecture/Motor Control - Drivers/Motor Control - Driver 0/FAULT_LED
- net Net-(LED1101-A) renamed /Project Architecture/Motor Control - Drivers/Motor Control - Driver 1/FAULT_LED
- net Net-(LED1201-A) renamed /Project Architecture/Motor Control - Drivers/Motor Control - Driver 2/FAULT_LED
- net Net-(LED1301-A) renamed /Project Architecture/Motor Control - Drivers/Motor Control - Driver 3/FAULT_LED
- net Net-(LED1401-A) renamed /Project Architecture/Motor Control - Drivers/Motor Control - Driver 4/FAULT_LED
- net Net-(LED1501-A) renamed /Project Architecture/Motor Control - Drivers/Motor Control - Driver 5/FAULT_LED
- net Net-(LED1601-A) renamed /Project Architecture/Motor Control - Drivers/Motor Control - Driver 6/FAULT_LED
- net Net-(LED1701-A) renamed /Project Architecture/Motor Control - Drivers/Motor Control - Driver 7/FAULT_LED
- net Net-(LED1801-A) renamed /Project Architecture/Motor Control - Drivers/Motor Control - Driver 8/FAULT_LED
- net Net-(LED1901-A) renamed /Project Architecture/Motor Control - Drivers/Motor Control - Driver 9/FAULT_LED
- net Net-(LED2001-A) renamed /Project Architecture/Motor Control - Drivers/Motor Control - Driver 10/FAULT_LED
- net Net-(LED2101-A) renamed /Project Architecture/Motor Control - Drivers/Motor Control - Driver 11/FAULT_LED
- net Net-(LED2201-A) renamed /Project Architecture/Motor Control - Drivers/Motor Control - Driver 12/FAULT_LED
- net Net-(LED2301-A) renamed /Project Architecture/Motor Control - Drivers/Motor Control - Driver 13/FAULT_LED
- net Net-(LED2401-A) renamed /Project Architecture/Motor Control - Drivers/Motor Control - Driver 14/FAULT_LED
- net Net-(LED2501-A) renamed /Project Architecture/Motor Control - Drivers/Motor Control - Driver 15/FAULT_LED
- net Net-(LED2601-A) renamed /Project Architecture/Motor Control - Drivers/Motor Control - Driver 16/FAULT_LED
- net Net-(LED2701-A) renamed /Project Architecture/Motor Control - Drivers/Motor Control - Driver 17/FAULT_LED
- net Net-(LED501-K) renamed /Project Architecture/Power - Battery Management/CHARGE_LED
- net Net-(R401-Pad1) renamed /Project Architecture/MCU - Unit/BOOT0_B
- D401 pad 1: /Project Architecture/MCU - Unit/USART1_RX -> /Project Architecture/MCU - Unit/USART1_RX_C
- D401 pad 3: /Project Architecture/MCU - Unit/USART1_TX -> /Project Architecture/MCU - Unit/USART1_RX_C
- J401 pad 2: /Project Architecture/MCU - Unit/USART1_TX -> /Project Architecture/MCU - Unit/USART1_RX_C
- J401 pad 3: /Project Architecture/MCU - Unit/USART1_RX -> /Project Architecture/MCU - Unit/USART1_RX_C
- R403 pad 1: Net-(U401A-PA9) -> /Project Architecture/MCU - Unit/USART1_TX
- R403 pad 2: /Project Architecture/MCU - Unit/USART1_TX -> /Project Architecture/MCU - Unit/USART1_RX_C
- R404 pad 1: Net-(U401A-PA10) -> /Project Architecture/MCU - Unit/USART1_RX
- R404 pad 2: /Project Architecture/MCU - Unit/USART1_RX -> /Project Architecture/MCU - Unit/USART1_RX_C
- U401 pad 1: unconnected-(U401A-PA2-Pad1) -> /Project Architecture/MCU - Unit/EN2
- U401 pad 18: unconnected-(U401A-PB7-Pad18) -> /Project Architecture/MCU - Unit/BUTTON1
- U401 pad 19: unconnected-(U401A-PB5-Pad19) -> /Project Architecture/MCU - Unit/BUTTON2
- U401 pad 2: unconnected-(U401A-PA1-Pad2) -> /Project Architecture/MCU - Unit/BAT_SENSE
- U401 pad 20: unconnected-(U401A-PB4-Pad20) -> /Project Architecture/MCU - Unit/BUTTON3
- U401 pad 22: unconnected-(U401A-PC10-Pad22) -> /Project Architecture/MCU - Unit/BUTTON4
- U401 pad 28: Net-(U401A-PA10) -> /Project Architecture/MCU - Unit/USART1_RX
- U401 pad 3: unconnected-(U401A-PA0-Pad3) -> /Project Architecture/MCU - Unit/BAT_SENSE_EN
- U401 pad 51: Net-(U401A-PA9) -> /Project Architecture/MCU - Unit/USART1_TX
- U401 pad 56: unconnected-(U401A-PA3-Pad56) -> /Project Architecture/MCU - Unit/EN1
- U401 pad 7: unconnected-(U401A-PC3-Pad7) -> /Project Architecture/MCU - Unit/DIN_3V3
- U401 pad 77: /Project Architecture/MCU - Unit/EN1 -> unconnected-(U401A-PD10-Pad77)
- U401 pad 8: unconnected-(U401A-PC2-Pad8) -> /Project Architecture/MCU - Unit/5V_ENABLE
- U401 pad 82: /Project Architecture/MCU - Unit/EN2 -> unconnected-(U401A-PD11-Pad82)
Routing:
- net /Project Architecture/Power - Battery Management/+VBAT: track 0.00 -> 4.16 mm
- net /Project Architecture/Motor Control - Drivers/OUT1_11: track 0.00 -> 4.14 mm
- net Net-(IC2601-IPROPI): track 0.00 -> 3.78 mm
- net /Project Architecture/Motor Control - Drivers/OUT1_16: track 0.00 -> 3.70 mm
- net /Project Architecture/Motor Control - Drivers/OUT2_16: track 0.00 -> 3.66 mm
- net /Project Architecture/MCU - Unit/nFault16: track 0.00 -> 3.28 mm
- net GND: track 0.00 -> 2.66 mm
- net /Project Architecture/Motor Control - Drivers/Motor Control - Driver 16/RC_OUT: track 0.00 -> 2.65 mm
- net /Project Architecture/Motor Control - Drivers/Motor Control - Driver 16/FAULT_LED: track 0.00 -> 1.63 mm
- added copper zone on B.Cu, net GND
- added copper zone on F.Cu, net GND
- added copper zone on In1.Cu, net GND
- added copper zone on In2.Cu, net GND
- added copper zone on In3.Cu, net GND
- added copper zone on In4.Cu, net GND
Other:
- outline, holes or cut-outs redrawn
