File: Power_Path_Generation.kicad_sch (KiCad schematic)
At the start: 11 parts, among them Q701 PMOS SI2365EDS-T1-GE3, U701 TPS3839G33DQNR, U702 TPS7A0233DBVR

Commit message: Finished layout, only cleaning left
Parts:
- U701: footprint Package_SON:Texas_X2SON-4_1x1mm_P0.65mm -> 0_Plume:Texas_X2SON-4_1x1mm_P0.65mm
- renumbered C704 to C702
Changed lines of the file:
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@@
 			"AAAAAAAAAAAAAAAAAAAAAAAAAAAAAAAAAAAAAAAAAAAAAAAAAAAAAAAAAAAAAAAAAAAAAAAAAAAA"
 			"AAAAAAAAAAAAAAAAAAAAAAAAAAAAAAAAAAAAAAAAAAAAAAAAAAAAAAAAAAAAAAAAAAAAAAAAAAAA"
+			"AAAAAAAAAAAAAAAAAAAAAAAAAAAAAAAAAAAAAAAAAAAAAAAAAAAAAAAAAAAACAAAAAAAAACAqrgI"
+			"AAAAABFnfgUAAAAAjg4AAAAAAADQulhYAQAAAGC7WFgBAAAAAAAAAAAAAABgCbEIAAAAABFnfgUA"
+			"AAAAjw4AAAAAAAAAu1hYAQAAAKC6WFgBAAAACAAAAAAAAABgCbEIAAAAANHRZwUAAAAAkA4AAAAA"
+			"AAAwu1hYAQAAANC6WFgBAAAAAAAAAAAAAADw2bQIAAAAANHRZwUAAAAAkQ4AAAAAAABgu1hYAQAA"
+			"AAC7WFgBAAAAAAAAAAAAAACAqrgIAAAAANHRZwUAAAAAkg4AAAAAAACgulhYAQAAADC7WFgBAAAA"
+			"BAAAAAAAAADw2bQIAAAAAKE3ggUAAAAAkw4AAAAAAADAu1hYAQAAAFC8WFgBAAAACAAAAAAAAADw"
+			"2bQIAAAAAIGWegUAAAAAlA4AAAAAAADwu1hYAQAAAJC7WFgBAAAAAAAAAAAAAAAAGMYIAAAAAIGW"
+			"egUAAAAAlQ4AAAAAAAAgvFhYAQAAAMC7WFgBAAAABAAAAAAAAAAAGMYIAAAAABFnfgUAAAAAlg4A"
+			"AAAAAABQvFhYAQAAAPC7WFgBAAAAAAAAAAAAAAAAGMYIAAAAAKE3ggUAAAAAlw4AAAAAAACQu1hY"
+			"AQAAACC8WFgBAAAAAAAAAAAAAABgCbEIAAAAABFnfgUAAAAAmA4AAAAAAACwvFhYAQAAAEC9WFgB"
+			"AAAAAAAAAAAAAACAqrgIAAAAABFnfgUAAAAAmQ4AAAAAAADgvFhYAQAAAIC8WFgBAAAABAAAAAAA"
+			"AACAqrgIAAAAAFH8lAUAAAAAmg4AAAAAAAAQvVhYAQAAALC8WFgBAAAAAAAAAAAAAADw2bQIAAAA"
+			"AFH8lAUAAAAAmw4AAAAAAABAvVhYAQAAAOC8WFgBAAAAAAAAAAAAAABgCbEIAAAAAFH8lAUAAAAA"
+			"nA4AAAAAAACAvFhYAQAAABC9WFgBAAAACAAAAAAAAADw2bQIAAAAAIGWegUAAAAAnQ4AAAAAAACg"
+			"vVhYAQAAADC+WFgBAAAABAAAAAAAAADw2bQIAAAAAKE3ggUAAAAAng4AAAAAAADQvVhYAQAAAHC9"
+			"WFgBAAAAAAAAAAAAAADgm6MIAAAAAKE3ggUAAAAAnw4AAAAAAAAAvlhYAQAAAKC9WFgBAAAACAAA"
+			"AAAAAADgm6MIAAAAABFnfgUAAAAAoA4AAAAAAAAwvlhYAQAAANC9WFgBAAAAAAAAAAAAAADgm6MI"
+			"AAAAAIGWegUAAAAAoQ4AAAAAAABwvVhYAQAAAAC+WFgBAAAAAAAAAAAAAACAqrgIAAAAAFFrRAUA"
+			"AAAAog4AAAAAAACQvlhYAQAAACC/WFgBAAAAAAAAAAAAAABgCbEIAAAAAAAAAAAAAAAAAAAAAAAA"
+			"AAAAAAAAAAAAAAAAAAAAAAAAAAAAAAAAAAAAAAAAAAAAAAAAAAAAAAAAAAAAAAAAAAAAAAAAAAAA"
+			"AAAAAAAAAAAAAAAAAAAAAAAAAAAAAAAAAAAAAAAAAAAAAAAAAAAAAAAAAAAAAAAAAAAAAAAAAAAA"
+			"AAAAAAAAAAAAAAAAAAAAAAAAAAAAAAAAAAAAAAAAAAAAAAAAAAAAAAAAAAAAAAAAAAAAAAAAAAAA"
+			"AAAAAAAAAAAAAAAAAAAAAAAAAAAAAAAAAAAAAAAAAAAAAAAAAAAAAAAAAAAAAAAAAAAAAAAAAAAA"
+			"AAAAAAAAAAAAAAAAAAAAAAAAAAAAAAAAAAAAAAAAAAAAAAAAAAAAAAAAAAAAAAAAAAAAAAAAAAAA"
+			"AAAAAAAAAAAAAAAAAAAAAAAAAAAAAAAAAAAAAAAAAAAAAAAAAAAAAAAAAAAAAAAAAAAAAAAAAAAA"
+			"AAAAAAAAAAAAAAAAAAAAAAAAAAAAAAAAAAAAAAAAAAAAAAAAAAAAAAAAAAAAAAAAAAAAAAAAAAAA"
+			"AAAAAAAAAAAAAAAAAAAAAAAAAAAAAAAAAAAAAAAAAAAAAAAAAAAAAAAAAAAAAAAAAAAAAAAAAAAA"
+			"AAAAAAAAAAAAAAAAAAAAAAAAAAAAAAAAAAAAAAAAAAAAAAAAAAAAAAAAAAAAAAAAAAAAAAAAAAAA"
+			"AAAAAAAAAAAAAAAAAAAAAAAAAAAAAAAAAAAAAAAAAAAAAAAAAAAAAAAAAAAAAAAAAAAAAAAAAAAA"
+			"AAAAAAAAAAAAAAAAAAAAAAAAAAAAAAAAAAAAAAAAAAAAAAAAAAAAAAAAAAAAAAAAAAAAAAAAAAAA"
+			"AAAAAAAAAAAAAAAAAAAAAAAAAAAAAAAAAAAAAAAAAAAAAAAAAAAAAAAAAAAAAAAAAAAAAAAAAAAA"
+			"AAAAAAAAAAAAAAAAAAAAAAAAAAAAAAAAAAAAAAAAAAAAAAAAAAAAAAAAAAAAAAAAAAAAAAAAAAAA"
+			"AAAAAAAAAAAAAAAAAAAAAAAAAAAAAAAAAAAAAAAAAAAAAAAAAAAAAAAAAAAAAAAAAAAAAAAAAAAA"
+			"AAAAAAAAAAAAAAAAAAAAAAAAAAAAAAAAAAAAAAAAAAAAAAAAAAAAAAAAAAAAAAAAAAAAAAAAAAAA"
+			"AAAAAAAAAAAAAAAAAAAAAAAAAAAAAAAAAAAAAAAAAAAAAAAAAAAAAAAAAAAAAAAAAAAAAAAAAAAA"
+			"AAAAAAAAAAAAAAAAAAAAAAAAAAAAAAAAAAAAAAAAAAAAAAAAAAAAAAAAAAAAAAAAAAAAAAAAAAAA"
 			"AAAAAAAAAAAAAAAAAAAAAAAAAAAAAAAAAAAAAAAAAAAAAAAAAAAAAAAAAA=="
 		)
@@
 			"NTJjVjhZTUJCQTQ1N3dMcGUxcFp3Q0JBQUtHQ1RSc1VFK0dEeG1ndmFwNTg5K1RqNWQrcG4yZDBh"
 			"T0dTSzJzVE8zcnNBQUNDQ0FRTm9IUUIvUlV3NFlOSFNyejVzMkx1WGV2enB3cFo1NTVac3pIOGVz"
-			"QTZtcHhPM2Z1bEQvY2ZiZTg4Y1lidnBSUi9PcDZXVlpZN3hvcjlEaHc0RUJwMXF5WkwvVVVMWXA="
+			"QTZtcHhPM2Z1bEQvY2ZiZTg4Y1lidnBSUi9PcDZXVlpZN3hvcjlEaHc0RUJwMXF5WkwvVVVMWXD/"
+			"////////////////////////////////////////////////////////////////////////////"
+			"////////////////////////////////////////////////////////////////////////////"
+			"////////////////////////////////////////////////////////////////////////////"
+			"////////////////////////////////////////////////////////////////////////////"
+			"////////////////////////////////////////////////////////////////////////////"
+			"////////////////////////////////////////////////////////////////////////////"
+			"////////////////////////////////////////////////////////////////////////////"
+			"////////////////////////////////////////////////////////////////////////////"
+			"////////////////////////////////////////////////////////////////////////////"
+			"////////////////////////////////////////////////////////////////////////////"
+			"////////////////////////////////////////////////////////////////////////////"
+			"////////////////////////////////////////////////////////////////////////////"
+			"////////////////////////////////////////////////////////////////////////////"
+			"////////////////////////////////////////////////////////////////////////////"
+			"////////////////////////////////////////////////////////////////////////////"
+			"////////////////////////////////////////////////////////////////////////////"
+			"////////////////////////////////////////////////////////////////////////////"
+			"/////////////////////////////////////////////////////////////////////////wAA"
+			"AAAAAAAAAAAAAAAAAAAAAAAAAAAAAAAAAAAAAAAAAAAAAAAAAAAAAAAAAAAAAAAAAAAAAAAAAAAA"
+			"AAAAAAAAAAAAAAAAAAAAAAAAAAAAAAAAAAAAAAAAAAAAAAAAAAAAAAAAAAAAAAAAAAAAAAAAAAAA"
+			"AAAAAAAAAAAAAAAAAAAAAAAAAAAAAAAAAAAAAAAAAAAAAAAAAAAAAAAAAAAAAAAAAAAAAAAAAAAA"
+			"AAAAAAAAAAAAAAAAAAAAAAAAAAAAAAAAAAAAAAAAAAAAAAAAAAAAAAAAAAAAAAAAAAAAAAAAAAAA"
+			"AAAAAAAAAAAAAAAAAAAAAAAAAAAAAAAAAAAAAAAAAAAAAAAAAAAAAAAAAAAAAAAAAAAAAAAAAAAA"
+			"AAAAAAAAAAAAAAAAAAAAAAAAAAAAAAAAAAAAAAAAAAAAAAAAAAAAAAAAAAAAAAAAAAAAAAAAAAAA"
+			"AAAAAAAAAAAAAAAAAAAAAAAAAAAAAAAAAAAAAAAAAAAAAAAAAAAAAAAAAAAAAAAAAAAAAAAAAAAA"
+			"AAAAAAAAAAAAAAAAAAAAAAAAAAAAAAAAAAAAAAAAAAAAAAAAAAAAAAAAAAAAAAAAAAAAAAAAAAAA"
+			"AAAAAAAAAAAAAAAAAAAAAAAAAAAAAAAAAAAAAAAAAAAAAAAAAAAAAAAAAAAAAAAAAAAAAAAAAAAA"
+			"AAAAAAAAAAAAAAAAAAAAAAAAAAAAAAAAAAAAAAAAAAAAAAAAAAAAAAAAAAAAAAAAAAAAAAAAAAAA"
+			"AAAAAAAAAAAAAAAAAAAAAAAAAAAAAAAAAAAAAAAAAAAAAAAAAAAAAAAAAAAAAAAAAAAAAAAAAAAA"
+			"AAAAAAAAAAAAAAAAAAAAAAAAAAAAAAAAAAAAAAAAAAAAAAAAAAAAAAAAAAAAAAAAAAAAAAAAAAAA"
+			"AAAAAAAAAAAAAAAAAAAAAAAAAAAAAAAAAAAAAAAAAAAAAAAAAAAAAAAAAAAAAAAAAAAAAAAAAAAA"
+			"AAAAAAAAAAAAAAAAAAAAAAAAAAAAAAAAAAAAAAAAAAAAAAAAAAAAAAAAAAAAAAAAAAAAAAAAAAAA"
+			"AAAAAAAAAAAAAAAAAAAAAAAAAAAAAAAAAAAAAAAAAAAAAAAAAAAAAAAAAAAAAAAAAAAAAAAAAAAA"
+			"AAAAAAAAAAAAAAAAAAAAAAAAAAAAAAAAAAAAAAAAAAAAAAAAAAAAAAAAAAAAAAAAAAAAAAAAAAAA"
+			"AAAAAAAAAAAAAAAAAAAAAAAAAAAAAAAAAAAAAAAAAAAAAAAAAAAAAAAAAAAAAAAAAAAAAAAAAAAA"
+			"AAAAAAAAAAAAAAAAAAAAAAAAAAAAAAAAAAAAAAAAAAAAAAAAAAAAAAAAAAAAAAAAAAAAAAAAAA=="
 		)
 	)
@@
 		(on_board yes)
 		(dnp no)
-		(property "Reference" "C704"
+		(property "Reference" "C702"
 			(at 160.274 113.03 0)
 			(effects
@@
 			(project "Plume"
 				(path "/0650c7a8-acba-429c-9f8e-eec0baf0bc1c/fede4c36-00cc-4d3d-b71c-5243ba232202/1d8841d3-b2be-4035-b859-53b06135dc6a"
-					(reference "C704")
+					(reference "C702")
 					(unit 1)
 				)
@@
 			)
 		)
-		(property "Footprint" "Package_SON:Texas_X2SON-4_1x1mm_P0.65mm"
+		(property "Footprint" "0_Plume:Texas_X2SON-4_1x1mm_P0.65mm"
 			(at 166.37 110.49 0)
 			(effects

Commit message: Finished cleaning routing, removed errors, cleaned shematics, added pictures and other improvements
Other:
- note added: "SOT-23-5 2.9mm×2.8mm"
