File: Power - Sequencing.kicad_sch (KiCad schematic)
At the start: 0 parts

Commit message: Cleaned repo, cleaned and exported shematic, advanced rough layout
Other:
- note added: "TO BE TESTED"
Changed lines of the file:
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@@
 	(title_block
 		(title "Power - Sequencing")
-		(date "2025-02-16")
+		(date "2025-04-05")
 		(rev "${REVISION}")
 		(company "${COMPANY}")
@@
 			)
 			(justify left bottom)
+		)
+	)
+	(text "TO BE TESTED"
+		(exclude_from_sim no)
+		(at 72.136 145.542 0)
+		(effects
+			(font
+				(size 7.62 7.62)
+				(thickness 0.762)
+				(bold yes)
+				(color 255 0 0 1)
+			)
 		)
 	)
@@
 		)
 	)
-	(text_box "Tip: you can set NetClass Colors for different voltage rails in File → Schematic Setup → Project → Net Classes"
-		(exclude_from_sim no)
-		(at 11.43 212.09 0)
-		(size 173.99 6.35)
-		(margins 1.9049 1.9049 1.9049 1.9049)
-		(stroke
-			(width -0.0001)
-			(type default)
-		)
-		(fill
-			(type none)
-		)
-		(effects
-			(font
-				(size 2.54 2.54)
-				(thickness 0.381)
-				(bold yes)
-				(color 0 0 0 1)
-			)
-			(justify right top)
-		)
-	)
